File: plate/plate.kicad_pcb (KiCad board)
At the start: 2 copper layers, 0 parts

Commit message: plate edge cuts
Other:
- board outline added: 266.7 x 98.7 mm

Commit message: plate fill
Routing:
- added copper zone on B.Cu, net (none)
- added copper zone on F.Cu, net (none)
Changed lines of the file:
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@@
     (47 F.CrtYd user)
     (48 B.Fab user hide)
-    (49 F.Fab user)
+    (49 F.Fab user hide)
   )
   (setup
@@
   (gr_line (start 189.213216 156.2237) (end 203.213916 156.2237) (layer Edge.Cuts) (width 0.05))
   (gr_line (start 246.364916 213.37386) (end 260.363916 213.37386) (layer Edge.Cuts) (width 0.05))
+  (zone (net 0) (net_name "") (layer B.Cu) (hatch edge 0.508)
+    (connect_pads (clearance 0.508))
+    (min_thickness 0.254)
+    (fill yes (arc_segments 32) (thermal_gap 0.508) (thermal_bridge_width 0.508))
+    (polygon
+      (pts
+        (xy 410.82 154.94) (xy 409.856945 174.543428) (xy 406.977056 193.958064) (xy 402.208067 212.996935) (xy 395.595906 231.476686)
+        (xy 387.204252 249.219347) (xy 377.113922 266.054046) (xy 365.42209 281.818656) (xy 352.241356 296.361356) (xy 337.698656 309.54209)
+        (xy 321.934046 321.233922) (xy 305.099347 331.324252) (xy 287.356686 339.715906) (xy 268.876935 346.328067) (xy 249.838064 351.097056)
+        (xy 230.423428 353.976945) (xy 210.82 354.94) (xy 191.216572 353.976945) (xy 171.801936 351.097056) (xy 152.763065 346.328067)
+        (xy 134.283314 339.715906) (xy 116.540653 331.324252) (xy 99.705954 321.233922) (xy 83.941344 309.54209) (xy 69.398644 296.361356)
+        (xy 56.21791 281.818656) (xy 44.526078 266.054046) (xy 34.435748 249.219347) (xy 26.044094 231.476686) (xy 19.431933 212.996935)
+        (xy 14.662944 193.958064) (xy 11.783055 174.543428) (xy 10.82 154.94) (xy 11.783055 135.336572) (xy 14.662944 115.921936)
+        (xy 19.431933 96.883065) (xy 26.044094 78.403314) (xy 34.435748 60.660653) (xy 44.526078 43.825954) (xy 56.21791 28.061344)
+        (xy 69.398644 13.518644) (xy 83.941344 0.33791) (xy 99.705954 -11.353922) (xy 116.540653 -21.444252) (xy 134.283314 -29.835906)
+        (xy 152.763065 -36.448067) (xy 171.801936 -41.217056) (xy 191.216572 -44.096945) (xy 210.82 -45.06) (xy 230.423428 -44.096945)
+        (xy 249.838064 -41.217056) (xy 268.876935 -36.448067) (xy 287.356686 -29.835906) (xy 305.099347 -21.444252) (xy 321.934046 -11.353922)
+        (xy 337.698656 0.33791) (xy 352.241356 13.518644) (xy 365.42209 28.061344) (xy 377.113922 43.825954) (xy 387.204252 60.660653)
+        (xy 395.595906 78.403314) (xy 402.208067 96.883065) (xy 406.977056 115.921936) (xy 409.856945 135.336572)
+      )
+    )
+  )
+  (zone (net 0) (net_name "") (layer F.Cu) (hatch edge 0.508)
+    (connect_pads (clearance 0.508))
+    (min_thickness 0.254)
+    (fill yes (arc_segments 32) (thermal_gap 0.508) (thermal_bridge_width 0.508))
+    (polygon
+      (pts
+        (xy 410.82 154.94) (xy 409.856945 174.543428) (xy 406.977056 193.958064) (xy 402.208067 212.996935) (xy 395.595906 231.476686)
+        (xy 387.204252 249.219347) (xy 377.113922 266.054046) (xy 365.42209 281.818656) (xy 352.241356 296.361356) (xy 337.698656 309.54209)
+        (xy 321.934046 321.233922) (xy 305.099347 331.324252) (xy 287.356686 339.715906) (xy 268.876935 346.328067) (xy 249.838064 351.097056)
+        (xy 230.423428 353.976945) (xy 210.82 354.94) (xy 191.216572 353.976945) (xy 171.801936 351.097056) (xy 152.763065 346.328067)
+        (xy 134.283314 339.715906) (xy 116.540653 331.324252) (xy 99.705954 321.233922) (xy 83.941344 309.54209) (xy 69.398644 296.361356)
+        (xy 56.21791 281.818656) (xy 44.526078 266.054046) (xy 34.435748 249.219347) (xy 26.044094 231.476686) (xy 19.431933 212.996935)
+        (xy 14.662944 193.958064) (xy 11.783055 174.543428) (xy 10.82 154.94) (xy 11.783055 135.336572) (xy 14.662944 115.921936)
+        (xy 19.431933 96.883065) (xy 26.044094 78.403314) (xy 34.435748 60.660653) (xy 44.526078 43.825954) (xy 56.21791 28.061344)
+        (xy 69.398644 13.518644) (xy 83.941344 0.33791) (xy 99.705954 -11.353922) (xy 116.540653 -21.444252) (xy 134.283314 -29.835906)
+        (xy 152.763065 -36.448067) (xy 171.801936 -41.217056) (xy 191.216572 -44.096945) (xy 210.82 -45.06) (xy 230.423428 -44.096945)
+        (xy 249.838064 -41.217056) (xy 268.876935 -36.448067) (xy 287.356686 -29.835906) (xy 305.099347 -21.444252) (xy 321.934046 -11.353922)
+        (xy 337.698656 0.33791) (xy 352.241356 13.518644) (xy 365.42209 28.061344) (xy 377.113922 43.825954) (xy 387.204252 60.660653)
+        (xy 395.595906 78.403314) (xy 402.208067 96.883065) (xy 406.977056 115.921936) (xy 409.856945 135.336572)
+      )
+    )
+  )
 )
