File: plate/plate.kicad_pcb (KiCad board)
At the start: 2 copper layers, 266.7 x 98.7 mm, 0 parts

Commit message: idk
Other:
- board size 266.7 x 98.7 mm -> 266.7 x 100.3 mm
Changed lines of the file:
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@@
   (general
     (thickness 1.6)
-    (drawings 361)
+    (drawings 360)
     (tracks 0)
     (zones 0)
@@
     (uvia_dia 0.3)
     (uvia_drill 0.1)
+  )
+  (dimension 12.065 (width 0.15) (layer Dwgs.User)
+    (gr_text "12.065 mm" (at 85.695 124.1425 90) (layer Dwgs.User)
+      (effects (font (size 1 1) (thickness 0.15)))
+    )
+    (feature1 (pts (xy 100.965 118.11) (xy 86.408579 118.11)))
+    (feature2 (pts (xy 100.965 130.175) (xy 86.408579 130.175)))
+    (crossbar (pts (xy 86.995 130.175) (xy 86.995 118.11)))
+    (arrow1a (pts (xy 86.995 118.11) (xy 87.581421 119.236504)))
+    (arrow1b (pts (xy 86.995 118.11) (xy 86.408579 119.236504)))
+    (arrow2a (pts (xy 86.995 130.175) (xy 87.581421 129.048496)))
+    (arrow2b (pts (xy 86.995 130.175) (xy 86.408579 129.048496)))
   )
   (gr_line (start 189.2007 204.0612) (end 180.5259 204.0612) (layer Edge.Cuts) (width 0.05))
@@
     (arrow2b (pts (xy 91.44 117.475) (xy 92.566504 116.888579)))
   )
-  (dimension 98.679 (width 0.15) (layer Dwgs.User)
-    (gr_text "98.679 mm" (at 361.345 169.1005 270) (layer Dwgs.User)
-      (effects (font (size 1 1) (thickness 0.15)))
-    )
-    (feature1 (pts (xy 353.06 218.44) (xy 360.631421 218.44)))
-    (feature2 (pts (xy 353.06 119.761) (xy 360.631421 119.761)))
-    (crossbar (pts (xy 360.045 119.761) (xy 360.045 218.44)))
-    (arrow1a (pts (xy 360.045 218.44) (xy 359.458579 217.313496)))
-    (arrow1b (pts (xy 360.045 218.44) (xy 360.631421 217.313496)))
-    (arrow2a (pts (xy 360.045 119.761) (xy 359.458579 120.887504)))
-    (arrow2b (pts (xy 360.045 119.761) (xy 360.631421 120.887504)))
-  )
   (dimension 9.525 (width 0.15) (layer Dwgs.User)
     (gr_text "9.525 mm" (at 96.2025 221.645) (layer Dwgs.User)
@@
     (arrow2b (pts (xy 100.965 220.345) (xy 99.838496 220.931421)))
   )
-  (dimension 86.614 (width 0.15) (layer Dwgs.User)
-    (gr_text "86.614 mm" (at 86.965 163.068 90) (layer Dwgs.User)
-      (effects (font (size 1 1) (thickness 0.15)))
-    )
-    (feature1 (pts (xy 100.965 119.761) (xy 87.678579 119.761)))
-    (feature2 (pts (xy 100.965 206.375) (xy 87.678579 206.375)))
-    (crossbar (pts (xy 88.265 206.375) (xy 88.265 119.761)))
-    (arrow1a (pts (xy 88.265 119.761) (xy 88.851421 120.887504)))
-    (arrow1b (pts (xy 88.265 119.761) (xy 87.678579 120.887504)))
-    (arrow2a (pts (xy 88.265 206.375) (xy 88.851421 205.248496)))
-    (arrow2b (pts (xy 88.265 206.375) (xy 87.678579 205.248496)))
-  )
   (dimension 12.065 (width 0.15) (layer Dwgs.User)
     (gr_text "12.065 mm" (at 86.965 212.4075 270) (layer Dwgs.User)
@@
   (gr_line (start 358.139916 215.899807) (end 91.44 215.899807) (layer F.Fab) (width 0.05))
   (gr_line (start 358.139916 120.65) (end 358.139916 215.899807) (layer F.Fab) (width 0.05))
-  (gr_line (start 96.52 119.761) (end 353.06 119.761) (layer Edge.Cuts) (width 0.05))
+  (gr_line (start 96.52 118.11) (end 353.06 118.11) (layer Edge.Cuts) (width 0.05))
   (gr_arc (start 353.06 213.36) (end 353.06 218.44) (angle -90) (layer Edge.Cuts) (width 0.05))
-  (gr_arc (start 96.52 124.841) (end 96.52 119.761) (angle -90) (layer Edge.Cuts) (width 0.05))
+  (gr_arc (start 96.52 123.19) (end 96.52 118.11) (angle -90) (layer Edge.Cuts) (width 0.05))
   (gr_arc (start 96.52 213.36) (end 91.44 213.36) (angle -90) (layer Edge.Cuts) (width 0.05))
   (gr_line (start 96.52 218.44) (end 353.06 218.44) (layer Edge.Cuts) (width 0.05))
-  (gr_line (start 358.14 213.36) (end 358.14 124.841) (layer Edge.Cuts) (width 0.05))
-  (gr_arc (start 353.06 124.841) (end 358.14 124.841) (angle -90) (layer Edge.Cuts) (width 0.05))
-  (gr_line (start 91.44 124.841) (end 91.44 213.36) (layer Edge.Cuts) (width 0.05))
+  (gr_line (start 358.14 213.36) (end 358.14 123.19) (layer Edge.Cuts) (width 0.05))
+  (gr_arc (start 353.06 123.19) (end 358.14 123.19) (angle -90) (layer Edge.Cuts) (width 0.05))
+  (gr_line (start 91.44 123.19) (end 91.44 213.36) (layer Edge.Cuts) (width 0.05))
   (zone (net 0) (net_name "") (layer B.Cu) (hatch edge 0.508)
     (connect_pads (clearance 0.508))

Commit message: i2c fin
Parts:
- added REF**: MountingHole_2.2mm_M2, MountingHole:MountingHole_2.2mm_M2, F.Cu at (92.3, 215.3)
- added REF**: MountingHole_2.2mm_M2, MountingHole:MountingHole_2.2mm_M2, F.Cu at (357.5, 215.0)
- added REF**: MountingHole_2.2mm_M2, MountingHole:MountingHole_2.2mm_M2, F.Cu at (357.3, 121.3)
- added REF**: MountingHole_2.2mm_M2, MountingHole:MountingHole_2.2mm_M2, F.Cu at (92.1, 121.5)
Routing:
- removed copper zone on B.Cu, net (none)
- removed copper zone on F.Cu, net (none)
Other:
- board size 266.7 x 100.3 mm -> 271.8 x 100.3 mm

Commit message: copper pour filling, mounting m2 holes pass 1
Parts:
- removed the REF** at (92.3, 215.3)
- removed the REF** at (357.5, 215.0)
- removed the REF** at (357.3, 121.3)
- removed the REF** at (92.1, 121.5)
- added REF**: MountingHole_2.2mm_M2, MountingHole:MountingHole_2.2mm_M2, F.Cu at (186.7, 184.8)
- added REF**: MountingHole_2.2mm_M2, MountingHole:MountingHole_2.2mm_M2, F.Cu at (110.5, 165.7)
- added REF**: MountingHole_2.2mm_M2, MountingHole:MountingHole_2.2mm_M2, F.Cu at (110.5, 127.6)
- added REF**: MountingHole_2.2mm_M2, MountingHole:MountingHole_2.2mm_M2, F.Cu at (110.5, 203.8)
- added REF**: MountingHole_2.2mm_M2, MountingHole:MountingHole_2.2mm_M2, F.Cu at (262.9, 184.8)
- added REF**: MountingHole_2.2mm_M2, MountingHole:MountingHole_2.2mm_M2, F.Cu at (186.7, 127.6)
- added REF**: MountingHole_2.2mm_M2, MountingHole:MountingHole_2.2mm_M2, F.Cu at (148.6, 158.8)
- added REF**: MountingHole_2.2mm_M2, MountingHole:MountingHole_2.2mm_M2, F.Cu at (301.0, 158.8)
- added REF**: MountingHole_2.2mm_M2, MountingHole:MountingHole_2.2mm_M2, F.Cu at (262.9, 127.6)
- added REF**: MountingHole_2.2mm_M2, MountingHole:MountingHole_2.2mm_M2, F.Cu at (339.1, 165.7)
- added REF**: MountingHole_2.2mm_M2, MountingHole:MountingHole_2.2mm_M2, F.Cu at (339.1, 127.6)
- added REF**: MountingHole_2.2mm_M2, MountingHole:MountingHole_2.2mm_M2, F.Cu at (339.1, 203.8)

Commit message: plate resize
Other:
- board size 271.8 x 100.3 mm -> 271.8 x 103.6 mm
- net class Default removed
