File: keeb/keeb.kicad_pcb (KiCad board)
At the start: 2 copper layers, 266.7 x 100.3 mm, 161 parts, among them J101 AVR-ISP-6, J103 AudioJack4, J104 AudioJack4, SW101 SW_Push, SW102 SW_Push, SW103 SW_Push, SW104 SW_Push, SW105 SW_Push, SW106 SW_Push, SW107 SW_Push, SW108 SW_Push, SW109 SW_Push, SW110 SW_Push, SW111 SW_Push, SW112 SW_Push, SW113 SW_Push, SW114 SW_Push, SW115 SW_Push, SW116 SW_Push, SW117 SW_Push, SW118 SW_Push, SW119 SW_Push, SW120 SW_Push, SW121 SW_Push, SW122 SW_Push, SW123 SW_Push, SW124 SW_Push, SW125 SW_Push, SW126 SW_Push, SW127 SW_Push, SW128 SW_Push, SW129 SW_Push, SW130 SW_Push, SW131 SW_Push, SW132 SW_Push, SW133 SW_Push, SW134 SW_Push, SW135 SW_Push, SW136 SW_Push, SW137 SW_Push, SW138 SW_Push, SW139 SW_Push, SW140 SW_Push, SW141 SW_Push, SW142 SW_Push, SW143 SW_Push, SW144 SW_Push, SW145 SW_Push, SW146 SW_Push, SW147 SW_Push, SW148 SW_Push, SW149 SW_Push, SW150 SW_Push, SW151 SW_Push, SW152 SW_Push, SW153 SW_Push, SW154 SW_Push, SW155 SW_Push, SW156 SW_Push, SW157 SW_Push, SW158 SW_Push, SW159 SW_Push, SW160 SW_Push, SW161 SW_Push, SW162 SW_Push, SW163 SW_Push, SW164 SW_Push, SW165 SW_Push, SW166 SW_Push, SW167 SW_Push, U101 ATmega32U4-AU, Y101 16Mhz

Commit message: fixed f mask fp
Parts:
- renumbered J104 to I2C_L101, J103 to I2C_R101, USB-C to J102
Connections:
- J102 pad A8: (no net) -> Net-(J102-PadA8)
- J102 pad B8: (no net) -> Net-(J102-PadB8)
- U101 pad 36: (no net) -> Net-(U101-Pad36)
- U101 pad 42: (no net) -> Net-(U101-Pad42)

Commit message: silk cleanu
Parts:
- renumbered I2C_L101 to I2C_101, I2C_R101 to I2C_102

Commit message: copper pour filling, mounting m2 holes pass 1
Parts:
- added REF**: MountingHole_2.2mm_M2, MountingHole:MountingHole_2.2mm_M2, F.Cu at (286.4, 149.2)
- added REF**: MountingHole_2.2mm_M2, MountingHole:MountingHole_2.2mm_M2, F.Cu at (95.9, 156.2)
- added REF**: MountingHole_2.2mm_M2, MountingHole:MountingHole_2.2mm_M2, F.Cu at (95.9, 118.1)
- added REF**: MountingHole_2.2mm_M2, MountingHole:MountingHole_2.2mm_M2, F.Cu at (95.9, 194.3)
- added REF**: MountingHole_2.2mm_M2, MountingHole:MountingHole_2.2mm_M2, F.Cu at (134.0, 149.2)
- added REF**: MountingHole_2.2mm_M2, MountingHole:MountingHole_2.2mm_M2, F.Cu at (248.3, 118.1)
- added REF**: MountingHole_2.2mm_M2, MountingHole:MountingHole_2.2mm_M2, F.Cu at (172.1, 118.1)
- added REF**: MountingHole_2.2mm_M2, MountingHole:MountingHole_2.2mm_M2, F.Cu at (248.3, 175.3)
- added REF**: MountingHole_2.2mm_M2, MountingHole:MountingHole_2.2mm_M2, F.Cu at (172.1, 175.3)
- added REF**: MountingHole_2.2mm_M2, MountingHole:MountingHole_2.2mm_M2, F.Cu at (324.5, 156.2)
- added REF**: MountingHole_2.2mm_M2, MountingHole:MountingHole_2.2mm_M2, F.Cu at (324.5, 118.1)
- added REF**: MountingHole_2.2mm_M2, MountingHole:MountingHole_2.2mm_M2, F.Cu at (324.5, 194.3)
Routing:
- net GND: track 11.9 -> 16.1 mm
- added copper zone on B.Cu, net (none)
- added copper zone on F.Cu, net (none)

Commit message: sync
Routing:
- net Net-(D135-Pad2): vias 0 -> 1

Commit message: fix sw mod and left over routing cleaning
Parts:
- moved R110 77.6 mm to (342.3, 127.6), turned to 90 degrees
- moved R107 76.9 mm to (83.5, 124.5), turned to 0 degrees
- moved R109 75.6 mm to (337.5, 131.4)
- moved I2C_102 75.5 mm to (334.6, 128.0)
- moved I2C_101 75.2 mm to (85.7, 128.0)
- moved R108 73.5 mm to (80.4, 131.4)
Routing:
- net SCL: track 285.7 -> 352.1 mm, vias 5 -> 6
- net SDA: track 285.0 -> 342.1 mm, vias 4 -> 5
- net +5V: track 119.8 -> 130.6 mm, vias 12 -> 16
- net COL_0: track 234.2 -> 239.0 mm
- net COL_11: track 172.8 -> 168.8 mm
- net VBUS: track 7.32 -> 4.62 mm
- net GND: track 16.1 -> 18.4 mm, vias 266 -> 264
- net ~RESET: track 101.5 -> 103.6 mm
- net D+: track 72.9 -> 73.6 mm
- net ROW_4: track 255.0 -> 254.9 mm, vias 3 -> 1
- removed copper zone on B.Cu, net (none)
- removed copper zone on F.Cu, net (none)
- removed copper zone on B.Cu, net D+
- removed copper zone on B.Cu, net D-
Other:
- rule via_min_drill: 0.3 -> 0.2

Commit message: logo begin
Routing:
- net GND: track 18.4 -> 16.1 mm

Commit message: kicad 6 upgrade
Connections:
- net ~HWB renamed ~{HWB}
- net ~RESET renamed ~{RESET}
Other:
- net class Default removed
