File: keeb/keeb.kicad_pcb (KiCad board)
At the start: 2 copper layers, 268 x 105 mm, 162 parts, among them J101 AVR-ISP-6, J102 USB_C_Receptacle_USB2.0, SW101 SW_Push, SW102 SW_Push, SW103 SW_Push, SW104 SW_Push, SW105 SW_Push, SW106 SW_Push, SW107 SW_Push, SW108 SW_Push, SW109 SW_Push, SW110 SW_Push, SW111 SW_Push, SW112 SW_Push, SW113 SW_Push, SW114 SW_Push, SW115 SW_Push, SW116 SW_Push, SW117 SW_Push, SW118 SW_Push, SW119 SW_Push, SW120 SW_Push, SW121 SW_Push, SW122 SW_Push, SW123 SW_Push, SW124 SW_Push, SW125 SW_Push, SW126 SW_Push, SW127 SW_Push, SW128 SW_Push, SW129 SW_Push, SW130 SW_Push, SW131 SW_Push, SW132 SW_Push, SW133 SW_Push, SW134 SW_Push, SW135 SW_Push, SW136 SW_Push, SW137 SW_Push, SW138 SW_Push, SW139 SW_Push, SW140 SW_Push, SW141 SW_Push, SW142 SW_Push, SW143 SW_Push, SW144 SW_Push, SW145 SW_Push, SW146 SW_Push, SW147 SW_Push, SW148 SW_Push, SW149 SW_Push, SW150 SW_Push, SW151 SW_Push, SW152 SW_Push, SW153 SW_Push, SW154 SW_Push, SW155 SW_Push, SW156 SW_Push, SW157 SW_Push, SW158 SW_Push, SW159 SW_Push, SW160 SW_Push, SW161 SW_Push, SW162 SW_Push, SW163 SW_Push, SW164 SW_Push, SW165 SW_Push, SW166 SW_Push, SW167 SW_Push, U101 TPD2S017, U102 ATmega32U4-MU, Y101 16Mhz

Commit message: First Routing Pass Complete
Parts:
- moved C107 2.43 mm to (147.5, 101.0), turned to 0 degrees
Routing:
- net +5V: track 429.3 -> 190.9 mm, vias 14 -> 21
- net /MOSI: track 9.51 -> 21.0 mm, vias 0 -> 2
- net /SCLK: track 10.4 -> 19.7 mm
- net /MISO: track 8.70 -> 18.0 mm
- net /~{RESET}: track 9.18 -> 17.8 mm, vias 0 -> 2
- net GND: track 37.9 -> 42.0 mm, vias 250 -> 312
- net /UCAP: track 3.80 -> 6.33 mm
- net /COL_7: track 74.2 -> 76.5 mm
- net /COL_0: track 212.3 -> 214.2 mm
- net /COL_5: track 113.6 -> 113.0 mm
- added copper zone on B.Cu, net +5V
- added copper zone on F.Cu, net +5V

Commit message: LCSC part selected
Routing:
- net GND: track 42.0 -> 43.8 mm, vias 312 -> 317
- net VBUS: vias 1 -> 0

Commit message: route cleanup
Parts:
- moved C108 0.20 mm to (156.2, 111.7)
- moved C109 0.20 mm to (156.1, 108.7)
- moved Y101 0.20 mm to (155.0, 110.2)
Routing:
- net GND: track 43.8 -> 43.0 mm
