File: hardware/keeb/keeb.kicad_pcb (KiCad board)
At the start: 2 copper layers, 268 x 104 mm, 162 parts, among them J101 AVR-ISP-6, J102 USB_C_Receptacle_USB2.0, SW101 SW_Push, SW102 SW_Push, SW103 SW_Push, SW104 SW_Push, SW105 SW_Push, SW106 SW_Push, SW107 SW_Push, SW108 SW_Push, SW109 SW_Push, SW110 SW_Push, SW111 SW_Push, SW112 SW_Push, SW113 SW_Push, SW114 SW_Push, SW115 SW_Push, SW116 SW_Push, SW117 SW_Push, SW118 SW_Push, SW119 SW_Push, SW120 SW_Push, SW121 SW_Push, SW122 SW_Push, SW123 SW_Push, SW124 SW_Push, SW125 SW_Push, SW126 SW_Push, SW127 SW_Push, SW128 SW_Push, SW129 SW_Push, SW130 SW_Push, SW131 SW_Push, SW132 SW_Push, SW133 SW_Push, SW134 SW_Push, SW135 SW_Push, SW136 SW_Push, SW137 SW_Push, SW138 SW_Push, SW139 SW_Push, SW140 SW_Push, SW141 SW_Push, SW142 SW_Push, SW143 SW_Push, SW144 SW_Push, SW145 SW_Push, SW146 SW_Push, SW147 SW_Push, SW148 SW_Push, SW149 SW_Push, SW150 SW_Push, SW151 SW_Push, SW152 SW_Push, SW153 SW_Push, SW154 SW_Push, SW155 SW_Push, SW156 SW_Push, SW157 SW_Push, SW158 SW_Push, SW159 SW_Push, SW160 SW_Push, SW161 SW_Push, SW162 SW_Push, SW163 SW_Push, SW164 SW_Push, SW165 SW_Push, SW166 SW_Push, SW167 SW_Push, U101 TPD2S017, U102 ATmega32U4-MU, Y101 16Mhz

Commit message: final parts and LCSC bom
Parts:
- R107, R108: value 22 -> 22R
Changed lines of the file:
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@@
     (tags "resistor")
     (property "LCSC #" "C25092")
-    (property "LCSC Link" "https://www.lcsc.com/product-detail/Chip-Resistor---Surface-Mount_UNI-ROYALUniroyal-Elec-UNI-ROYALUniroyal-Elec-0402WGF220JTCE_C25092.html")
+    (property "LCSC Link" "https://lcsc.com/product-detail/Chip-Resistor---Surface-Mount_UNI-ROYALUniroyal-Elec-UNI-ROYALUniroyal-Elec-0402WGF220JTCE_C25092.html")
     (property "Sheetfile" "keeb.kicad_sch")
     (property "Sheetname" "")
@@
         (effects (font (size 1 1) (thickness 0.15)) (justify mirror))
     )
-    (fp_text value "22" (at 0 -1.17 270) (layer "B.Fab") hide
+    (fp_text value "22R" (at 0 -1.17 270) (layer "B.Fab") hide
         (effects (font (size 1 1) (thickness 0.15)) (justify mirror))
     )
@@
     (tags "capacitor")
     (property "LCSC #" "C15849")
-    (property "LCSC Link" "https://datasheet.lcsc.com/lcsc/1810261812_Samsung-Electro-Mechanics-CL10A105KB8NNNC_C15849.pdf")
+    (property "LCSC Link" "https://lcsc.com/product-detail/Multilayer-Ceramic-Capacitors-MLCC---SMD-SMT_Samsung-Electro-Mechanics-Samsung-Electro-Mechanics-CL10A105KB8NNNC_C15849.html")
     (property "Sheetfile" "keeb.kicad_sch")
     (property "Sheetname" "")
@@
     (tags "capacitor")
     (property "LCSC #" "C15849")
-    (property "LCSC Link" "https://datasheet.lcsc.com/lcsc/1810261812_Samsung-Electro-Mechanics-CL10A105KB8NNNC_C15849.pdf")
+    (property "LCSC Link" "https://lcsc.com/product-detail/Multilayer-Ceramic-Capacitors-MLCC---SMD-SMT_Samsung-Electro-Mechanics-Samsung-Electro-Mechanics-CL10A105KB8NNNC_C15849.html")
     (property "Sheetfile" "keeb.kicad_sch")
     (property "Sheetname" "")
@@
     (property "ki_description" "Atmel 6-pin ISP connector")
     (property "ki_keywords" "AVR ISP Connector")
-    (property "man#" "")
     (attr smd)
     (fp_text reference "J101" (at -2.54 3.81 270 unlocked) (layer "B.SilkS") hide
@@
     (tags "resistor")
     (property "LCSC #" "C25092")
-    (property "LCSC Link" "https://www.lcsc.com/product-detail/Chip-Resistor---Surface-Mount_UNI-ROYALUniroyal-Elec-UNI-ROYALUniroyal-Elec-0402WGF220JTCE_C25092.html")
+    (property "LCSC Link" "https://lcsc.com/product-detail/Chip-Resistor---Surface-Mount_UNI-ROYALUniroyal-Elec-UNI-ROYALUniroyal-Elec-0402WGF220JTCE_C25092.html")
     (property "Sheetfile" "keeb.kicad_sch")
     (property "Sheetname" "")
@@
         (effects (font (size 1 1) (thickness 0.15)) (justify mirror))
     )
-    (fp_text value "22" (at 0 -1.17 270) (layer "B.Fab") hide
-        (effects (font (size 1 1) (thickness 0.15)) (justify mirror))
-    )
+    (fp_text value "22R" (at 0 -1.17 270) (layer "B.Fab") hide
+        (effects (font (size 1 1) (thickness 0.15)) (justify mirror))
+    )

Commit message: fp pin1 cleanup and general route polish (focus on i2c)
Parts:
- moved R104 0.76 mm to (268.5, 158.2)
- moved R105 0.75 mm to (31.5, 161.8)
- moved R106 0.75 mm to (31.5, 158.2)
- moved R103 0.74 mm to (268.5, 161.8)
Routing:
- net +5V: track 181.9 -> 175.2 mm
- net /~{RESET}: track 17.5 -> 15.4 mm
- net GND: track 42.8 -> 40.9 mm, vias 333 -> 334
- net /CC1: track 1.81 -> 0.00 mm
- net /SCL: track 279.6 -> 280.5 mm
- net /SDA: track 271.9 -> 272.8 mm
- net Net-(D128-A): track 8.06 -> 7.51 mm
- added copper zone on B.Cu, net /CC1
- added copper zone on B.Cu, net /UCAP
- added copper zone on B.Cu, net /~{RESET}
